File: FPC2COR_PCB/FPC2COR_PCB.kicad_pcb (KiCad board)
At the start: 2 copper layers, 0 parts

Commit message: Add files via upload
Parts:
- added +FP: ~, MountingHole:MountingHole_2.2mm_M2_ISO7380_Pad, F.Cu at (125.8, 68.2)
- added B+: ~, MountingHole:MountingHole_2.2mm_M2_ISO7380_Pad, F.Cu at (125.8, 73.2)
- added C1: 1uF_0603_25V, Capacitor_THT:C_Disc_D5.0mm_W2.5mm_P2.50mm, F.Cu at (111.2, 66.5)
- added DI: ~, MountingHole:MountingHole_2.2mm_M2_ISO7380_Pad, F.Cu at (125.8, 62.8)
- added DZ1: 1N4746A, Diode_THT:D_DO-41_SOD81_P10.16mm_Horizontal, F.Cu at (103.0, 53.1)
- added DZ2: 1N4746A, Diode_THT:D_DO-41_SOD81_P10.16mm_Horizontal, F.Cu at (108.0, 53.1)
- added E: ~, MountingHole:MountingHole_2.2mm_M2_ISO7380_Pad, F.Cu at (125.8, 52.2)
- added FPC: ~, MountingHole:MountingHole_2.2mm_M2_ISO7380_Pad, F.Cu at (125.8, 57.5)
- added J1: V23333-Z0002-B049, TE_CONNECTIVITY:V23333-Z0002-B049, F.Cu at (90.0, 63.8)
- added JP1: JUP_P10mm, PCM_SL_Jumpers:JUP_P10mm, F.Cu at (106.8, 74.3)
- added Q1: 2N7000, Package_TO_SOT_THT:TO-92, F.Cu at (105.0, 69.1)
- added R1: 1M, Resistor_THT:R_Axial_DIN0207_L6.3mm_D2.5mm_P10.16mm_Horizontal, F.Cu at (115.0, 65.7)
- added R2: 1k, Resistor_THT:R_Axial_DIN0207_L6.3mm_D2.5mm_P10.16mm_Horizontal, F.Cu at (119.7, 65.7)
Routing:
- net +B: track 0.00 -> 53.5 mm
- net +FP: track 0.00 -> 40.7 mm
- net Net-(DZ1-K): track 0.00 -> 33.7 mm
- net Net-(DZ2-K): track 0.00 -> 33.4 mm
- net DI: track 0.00 -> 18.8 mm
- net FPC: track 0.00 -> 10.7 mm
- added copper zone on B.Cu, net E
Other:
- board outline added: 47.2 x 26.8 mm
