File: FPC2COR_PCB/FPC2COR_PCB.kicad_sch (KiCad schematic)
At the start: 8 parts, among them J1 V23333-Z0002-B049, Q1 2N7000

Commit message: Add files via upload
Parts:
- added H1, H2, H3, H4, H5: ~, MountingHole:MountingHole_2.2mm_M2_ISO7380_Pad, symbol Mechanical:MountingHole_Pad
- DZ1, DZ2: footprint PCM_Diode_SMD_Handsoldering_AKL:D_MiniMELF_Zener -> Diode_THT:D_DO-41_SOD81_P10.16mm_Horizontal
- Q1: footprint PCM_Package_TO_SOT_THT_AKL:TO-92_Inline_Wide_SGD -> Package_TO_SOT_THT:TO-92
Connections:
- net +B: now also H1.1
- net +FP: now also H2.1
- net DI: now also H3.1
- net E: now also H5.1
- net FPC: now also H4.1
